File: PCB/StepperServoCAN.kicad_sch (KiCad schematic)
At the start: 132 parts, among them J1 CAR, J2 Debug, J3 Motor, J4 Conn_01x06, Q1 AO3401A, Q2 2N7002, Q3 AO3401A, SW1 Rst, U1 STM32F103CBT6, U2 TLE5012B, U3 A4950, U4 A4950, U5 SN65HVD230, U6 LMV321, U7 LMV321, U8 TMAG5170-Q1, U9 ADMT4000BRUZAB-R7, Y1 16Mhz 9pF

Commit message: outline etc.
Parts:
- removed C14: 100n, Capacitor_SMD:C_0402_1005Metric, symbol Device:C_Small
- removed TP10, TP4, TP5, TP6, TP8, TP9: WirePad, TestPoint:TestPoint_Pad_2.0x2.0mm, symbol Connector:TestPoint
- removed U8: TMAG5170-Q1, Package_SO:VSSOP-8_3.0x3.0mm_P0.65mm, symbol Sensor_Magnetic:TMAG5170-Q1
- removed U9: ADMT4000BRUZAB-R7, TSSOP-24_4.4x7.8mm_P0.65mm, symbol ADMT4000:ADMT4000BRUZAB-R7
- added H7, H8: Nema23, MountingHole:MountingHole_3.2mm_M3_ISO14580_Pad_TopOnly, symbol Mechanical:MountingHole_Pad
- added J5: CAR, Connector_JST:JST_XH_B4B-XH-A_1x04_P2.50mm_Vertical, symbol Connector_Generic:Conn_01x04
- J1, J3: footprint Connector_JST_SMD:JST-S4B-XH-SM4-TB -> Connector_JST:JST_XH_B4B-XH-A_1x04_P2.50mm_Vertical
Connections:
- net +BATT: now also J5.1 (Pin_1); no longer J1.6 (Mount)
- net CAN_H: now also J5.3 (Pin_3)
- net CAN_L: now also J5.2 (Pin_2)
- net GND: now also H7.1, H8.1, J5.4 (Pin_4); no longer J1.5 (Mount), J3.5 (Mount), J3.6 (Mount)
Other:
- note removed: "To test ADMT4000: scrape silkscreen from footprint pads remove TLE5012B remove Q1&Q2 and short AUX_3.3 with 3.3V."
