File: PCB/StepperServoCAN.kicad_pcb (KiCad board)
At the start: 4 copper layers, 56 x 43.3 mm, 153 parts, among them J1 CAR, J2 Debug, J3 Motor, J4 Conn_01x06, Q1 AO3401A, Q2 2N7002, Q3 AO3401A, SW1 Rst, U1 STM32F103CBT6, U11 LV2842XLVDDCR, U2 TLE5012B, U3 A4950, U4 A4950, U5 SN65HVD230, U6 LMV321, U7 LMV321, U8 TMAG5170-Q1, U9 ADMT4000BRUZAB-R7, Y1 16Mhz 9pF

Commit message: outline etc.
Parts:
- removed the ? at (73.6, 87.8)
- removed C14: 100n, Capacitor_SMD:C_0402_1005Metric
- removed TP10, TP4, TP5, TP6, TP8, TP9: WirePad, TestPoint:TestPoint_Pad_2.0x2.0mm
- removed U8: TMAG5170-Q1, Package_SO:VSSOP-8_3.0x3.0mm_P0.65mm
- removed U9: ADMT4000BRUZAB-R7, Package_SO:TSSOP-24_4.4x7.8mm_P0.65mm
- added H7: Nema23, MountingHole:MountingHole_3.2mm_M3_ISO14580_Pad_TopOnly, F.Cu at (200.9, 29.4)
- added H8: Nema23, MountingHole:MountingHole_3.2mm_M3_ISO14580_Pad_TopOnly, F.Cu at (200.9, 60.4)
- added J5: CAR, Connector_JST:JST_XH_B4B-XH-A_1x04_P2.50mm_Vertical, B.Cu at (99.4, 48.6)
- D22: footprint Package_TO_SOT_SMD:SOT-323_SC-70 -> Package_TO_SOT_SMD:SOT-23
- J1, J3: footprint Connector_JST_SMD:JST-S4B-XH-SM4-TB -> Connector_JST:JST_XH_B4B-XH-A_1x04_P2.50mm_Vertical; moved to B.Cu
- moved J3 135.5 mm to (226.9, 37.9), turned to 90 degrees
- moved H2 128.9 mm to (169.9, 29.4)
- moved C11 125.4 mm to (185.9, 25.6), turned to 90 degrees
- moved C12 125.3 mm to (181.4, 24.9), turned to -90 degrees
- moved Y1 124.7 mm to (183.7, 25.7), turned to 0 degrees
- moved R4 123.0 mm to (181.4, 26.6), turned to -90 degrees
- moved J1 121.4 mm to (226.9, 59.4)
- moved R21 116.6 mm to (190.8, 34.9), turned to -90 degrees
- moved U1 115.6 mm to (183.4, 33.5), turned to -90 degrees
- moved C22 115.5 mm to (191.6, 35.9), turned to -90 degrees
- moved R22 114.1 mm to (190.2, 36.5), turned to 180 degrees
- moved TP1 113.5 mm to (199.8, 86.9), turned to -90 degrees
- moved C23 112.9 mm to (190.3, 37.5), turned to 0 degrees
- moved R19 112.3 mm to (189.1, 37.6), turned to -90 degrees
- moved R28 111.6 mm to (199.4, 88.5), turned to -90 degrees
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Routing:
- net GND: track 184.8 -> 0.00 mm, vias 273 -> 5
- net +3.3V: track 116.2 -> 3.52 mm
- net UART_RX: track 78.5 -> 0.00 mm, vias 3 -> 0
- net UART_TX: track 77.7 -> 0.00 mm, vias 3 -> 0
- net AUX_3.3: track 78.1 -> 2.43 mm, vias 4 -> 0
- net Net-(FB1-Pad1): track 56.8 -> 0.00 mm, vias 3 -> 0
- net DCDC_SHUTDOWN: track 45.6 -> 0.00 mm, vias 4 -> 0
- net /R30: track 36.4 -> 0.00 mm, vias 4 -> 0
- net Net-(U1-NRST): track 33.8 -> 0.00 mm, vias 4 -> 0
- net +3.3VA: track 33.6 -> 0.00 mm, vias 2 -> 0
- net +BATT: track 33.6 -> 0.00 mm, vias 17 -> 0
- net LSS_A: track 30.5 -> 0.00 mm, vias 8 -> 0
- net /AUX_ON: track 28.7 -> 0.00 mm, vias 3 -> 0
- net LSS_A_ADC: track 26.9 -> 0.00 mm, vias 2 -> 0
- net VBATT_ADC: track 26.0 -> 0.00 mm, vias 7 -> 0
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Other:
- board size 56 x 43.3 mm -> 235 x 50 mm
- board text removed: "+"
- board text removed: "-------------"
- board text removed: "-> Apply thermal paste"
- board text removed: "120 Ω"
- board text removed: "3.3v"
- board text removed: "<- Nema23 mounting ->"
- board text removed: "<test"
- board text removed: "A1"
- board text removed: "A1 A2 B1 B2 MOTOR"
- board text removed: "A2"
- board text removed: "AUX"
- board text removed: "B1"
- board text removed: "B2"
- board text removed: "CAN"
- board text removed: "CAN_H"
- board text removed: "CAN_L"
- board text removed: "F1"
- board text removed: "F2"
- board text removed: "G"
- board text removed: "G ________ En ________ 3.3 ________ RX SDA ________ TX SCL ________ G ________"
- board text removed: "GND"
- board text removed: "H"
- board text removed: "ID1"
- board text removed: "ID2"
- board text removed: "JLCJLCJLCJLC"
- board text removed: "L"
- board text removed: "Min supp: 8V (11V start) Max supp: 30V Combined RMS I: 3.3A"
- board text removed: "Nema17"
- board text removed: "Nema23"
- board text removed: "Protect caps from mechanical flex"
- board text removed: "SCK"
- board text removed: "SWD"
- board text removed: "StepperServoCAN v0.4"
- board text removed: "Vehicle"
- board text removed: "Vin"
- board text removed: "_______"
- board text removed: "________"
- board text removed: "___________ Debug"
- board text removed: "____________"
- board text removed: "_______________"
- board text removed: "__________________________"

Commit message: wip
Parts:
- removed ? (x2): JLCPCB_ToolingHole, part:JLCPCB_ToolingHole
- C27, ID1, ID2, J2, JP10, JP11, TP1, TP2: moved to B.Cu
- moved FB1 97.2 mm to (189.1, 22.1), turned to 90 degrees
- moved JP11 95.3 mm to (198.6, 36.1)
- moved R49 94.6 mm to (111.4, 39.9), turned to -90 degrees
- moved FB2 94.3 mm to (104.6, 41.9), turned to -90 degrees
- moved R48 93.4 mm to (109.9, 40.4), turned to 180 degrees
- moved D19 93.3 mm to (106.6, 45.4)
- moved JP10 92.8 mm to (201.4, 36.1), turned to -90 degrees
- moved R3 92.5 mm to (112.4, 39.9), turned to 90 degrees
- moved D18 91.9 mm to (107.1, 41.9), turned to 180 degrees
- moved C38 91.2 mm to (109.4, 41.9)
- moved R35 91.0 mm to (199.1, 41.4), turned to -90 degrees
- moved J2 89.9 mm to (185.6, 8.16), turned to 0 degrees
- moved R46 89.8 mm to (114.9, 42.4), turned to -90 degrees
- moved C37 89.8 mm to (108.9, 44.6), turned to -90 degrees
- moved R34 88.3 mm to (201.1, 41.4)
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Routing:
- net +BATT: track 0.00 -> 211.1 mm, vias 0 -> 3
- net CAN_L: track 2.57 -> 175.5 mm
- net CAN_H: track 2.54 -> 171.9 mm, vias 0 -> 2
- net VMOT: track 0.00 -> 74.1 mm, vias 0 -> 15
- net +3.3VA: track 0.00 -> 62.2 mm, vias 0 -> 4
- net AUX_3.3: track 2.43 -> 46.9 mm, vias 0 -> 5
- net VBATT_ADC: track 0.00 -> 41.2 mm, vias 0 -> 4
- net Net-(U1-NRST): track 0.00 -> 39.9 mm, vias 0 -> 2
- net PWM_B_IN2: track 0.00 -> 38.0 mm, vias 0 -> 2
- net PWM_B_IN1: track 0.00 -> 37.6 mm, vias 0 -> 2
- net LSS_B_ADC: track 0.00 -> 35.6 mm, vias 0 -> 2
- net Net-(U1-PC14): track 0.00 -> 33.3 mm, vias 0 -> 2
- net LSS_A_ADC: track 0.00 -> 31.7 mm, vias 0 -> 2
- net Net-(U1-PC13): track 0.00 -> 30.8 mm, vias 0 -> 2
- net PWM_A_IN1: track 0.00 -> 30.3 mm, vias 0 -> 2
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- added copper zone on In1.Cu, net +3.3V
- removed copper zone on F.Cu, net +3.3V
- removed copper zone on F.Cu, net +BATT
- removed copper zone on In1.Cu, net GND
- removed copper zone on In2.Cu, net GND
- removed copper zone on F.Cu, net LSS_B
- removed copper zone on F.Cu, net Net-(D20-K)
- removed copper zone on F.Cu, net VMOT
Other:
- outline, holes or cut-outs redrawn
